Commit message: added interial properties base in urdf

File: gym_aliengo/urdf/aliengo.urdf (robot description, URDF)
Before this commit: robot aliengo_description, 19 links, 18 joints
Links:
- link base: mass None -> 0.0

Commit message: changing urdf back, apparently that breaks things...

File: gym_aliengo/urdf/aliengo.urdf (robot description, URDF)
Before this commit: robot aliengo_description, 19 links, 18 joints
Links:
- link base: mass 0.0 -> None
